Commit message: been extremely hard at work on this project, and I am proud of the progress we have made. The changes in this commit include updates to various Dockerfiles, Python scripts, and configuration files that enhance the functionality and performance of our system.
All changes to the robot's code. Newest first.

- **ESP32s / micro-ROS:** The serial numbers need to go into the udev rule. Driving, IMU and battery have not been tested yet.
- **Colour calibration of the IMX219:** libcamera uses `uncalibrated.yaml`, and the image has a faint greenish or cyan cast. A colour matrix for the IMX219 will be evaluated outdoors on grass.
- **depth_fusion:** 90 ms per frame (82 ms of it for the model) is close to the limit at 10 FPS. Options: run image preprocessing in parallel with the NPU, or export the model at 800×608 instead of 800×800. The export has been passed on to the model-export thread.
- **Active learning:** Watch whether "Saved uncertain object" becomes less frequent now that the image is the right way up.
- **VPU:** It can only encode and decode video (H.264/H.265). It is reserved for live video in the app.
- **ROS 2 Lyrical** (Ubuntu 26.04 in the containers) is waiting for qai-appbuilder to become available for Python 3.14.

---

Merged to main (pull request #4).

- **Fixed:** the app received no telemetry. The backend only sent status when a ROS topic arrived from the ESP32s (battery, motors, rain). Without the micro-ROS agents, which are only started with `docker compose --profile esp32`, nothing was ever sent. This also affected CPU, Wi-Fi and calibration. Status is now sent at a fixed interval of every two seconds.
- Status is sent immediately when the app connects to `/ws`, instead of waiting for the next broadcast.
- RAM usage is now included under `system.memory` as `used_mb`, `total_mb` and `used_pct`, read from `/proc/meminfo`.
- Status is not built when no app is connected.

After `~/omnimow/app_backend/backend_node.py` has been updated:

```sh
cd ~/omnimow/system_setup && docker compose up -d --build app_backend
```

---

Merged to main (pull request #5, branch `tuning`). Fine-tuning of the test setup on the Radxa Dragon Q6A (rafaelwms Ubuntu 26.04, mainline kernel). All figures were measured on the board.

| | Before (test-setup) | After (tuning) |
|---|---|---|
| depth_fusion: AI obstacles with depth | 3–5 per second | 10 per second |
| Stereo node | approx. 13 FPS, 1 core for SGBM | 10 FPS (deliberate), 62–68 ms per frame |
| CPU, all containers | approx. 4.5 cores | approx. 3.4 cores |
| Field of view | approx. 44° (1080p crop of the sensor) | approx. 72° × 58° (full sensor) |
| Shortest stereo depth | 0.75 m | 0.28 m |
| Calibration, stereo RMS | 0.98 px | 0.68 px (baseline 59.8 mm) |
| AI input | 640×360 upscaled to 800×450, upside down | 800×600 without upscaling, correct orientation |
| Software ISP (debayer) | CPU, 12–25 ms per frame | Adreno GPU, 2–5 ms per frame |

- **depth_fusion only received 3–5 of ~13 frames per second.** Messages larger than about 512 KB were mostly lost between containers. The colour image is now sent as JPEG (`/stereo/left/image_rect_color/compressed`), and depth is sent as 16-bit millimetres at half resolution (320×240, 154 KB). The full-resolution 640×480 depth image was 614 KB. The raw colour image is only published when something subscribes to it.
- **depth_fusion picked the depth image by arrival.** It took the newest depth image instead of the one from the same stereo frame. It now selects the one with a matching timestamp among the last 5.
- **Stereo was blind at close range.** 64 disparities only gave depth from 0.75 m, even though the ground is in view from about 0.45 m. 96 disparities are now used, and together with the wide field of view this gives depth from 0.28 m.
- **The image was upside down.** The cameras are mounted upside down on the test rig. With `OMNIMOW_CAMERA_UPSIDE_DOWN=true`, both images are rotated 180° and the left and right cameras are swapped.
- **libcamera bug in the GPU ISP (patch 0002).** When the GPU downscaled the image, exposure and white balance were computed from the top-left corner only. The whole image is now used.
- **1080p mode actually ran the sensor at full resolution (3280×2464),** which limited the cameras to 15 FPS.
- **Calibration with the board in motion.** The cameras don't capture at exactly the same instant, so a moving board sits in different places in the left and right images. This made the stereo error almost twice each camera's own error (0.90 vs 0.45–0.53 px), and the baseline varied between 59.7 and 63.9 mm. A frame is now only captured when the board is still.

**ROS 2 transport**

- depth_fusion logs received frames and depth images per second, and how many of them find a matching depth image.

**Camera (stereo_vision)**

- The software ISP runs on the Adreno GPU (`LIBCAMERA_SOFTISP_MODE=gpu`, Mesa 25.2).
- The GPU scales the full sensor image directly to the requested size (`OMNIMOW_CAMERA_GPU_SCALE=true`). libcamera then selects the IMX219's binned 1640×1232 mode, which gives the full field of view, less noise and no 1080p conversion on the CPU. The camera size is 640×480 (4:3). Requires a new calibration.
- Camera frame rate is set directly on the sensor via vertical blanking (`OMNIMOW_CAMERA_FPS=30`). Without it, the binned mode runs at about 60 FPS. At 30 FPS, the left and right images in a pair are at most 17 ms apart.
- `OMNIMOW_CAMERA_UPSIDE_DOWN` for a camera pair mounted upside down.
- The AI gets its own, larger colour image (`OMNIMOW_AI_IMAGE_WIDTH=800`, i.e. 800×600) instead of the 640×360 stereo image upscaled 1.25×. It is rectified at full size and scaled down for stereo. The model's 800×800 input now has 25 % grey padding instead of 44 %.

**Stereo**

- SGBM uses multiple threads (`OMNIMOW_STEREO_MODE=3way`, `OMNIMOW_STEREO_THREADS=4`). This was about 4× faster in a test on another machine.
- The stereo computation runs in a worker thread while frames are being published.
- The stereo node processes at most `OMNIMOW_STEREO_FPS=10` frames per second. This also saves work in depth_fusion, SLAM and navigation.
- The log shows time per stage: rectify, publish, disparity wait, and depth+scan.

**Calibration**

- Rational lens model with 8 coefficients (`OMNIMOW_CALIB_MODEL=rational`) for the wide-angle lenses.
- A frame is only captured when the board is still (`OMNIMOW_CALIB_STILL_PX=0.5`).
- The final message also shows the RMS for each camera.
- Calibration can be recomputed from the saved image pairs without holding up the board again: `calibrate_stereo.py --images /calibration/samples`.

**depth_fusion**

- Masks from the 800×600 AI image are scaled to the depth image's size. The projection maps the pixels back into camera coordinates.

| Setting | Default | Meaning |
|---|---|---|
| `LIBCAMERA_SOFTISP_MODE` | `gpu` | Debayer on the GPU (`cpu` as fallback) |
| `OMNIMOW_CAMERA_GPU_SCALE` | `true` | The GPU scales the full sensor image. Requires a 4:3 size |
| `OMNIMOW_CAMERA_WIDTH` / `HEIGHT` | `640` / `480` | Camera size for stereo (was 640×360) |
| `OMNIMOW_CAMERA_FPS` | `30` | Camera frame rate, set on the sensor |
| `OMNIMOW_CAMERA_UPSIDE_DOWN` | `true` | The camera pair is mounted upside down (test rig) |
| `OMNIMOW_AI_IMAGE_WIDTH` | `800` | Width of the AI's colour image |
| `OMNIMOW_STEREO_NUM_DISPARITIES` | `96` | Shortest depth = focal length × baseline / disparities |
| `OMNIMOW_STEREO_MODE` | `3way` | SGBM mode |
| `OMNIMOW_STEREO_FPS` | `10` | Maximum stereo frames per second |
| `OMNIMOW_STEREO_THREADS` | `4` | Number of OpenCV threads |
| `OMNIMOW_CALIB_MODEL` | `rational` | Lens model: `rational` or `standard` |
| `OMNIMOW_CALIB_STILL_PX` | `0.5` | How still the board must be before a frame is captured |

- **A new stereo calibration is required.** Image size, sensor mode and orientation have changed. Delete `/opt/omnimow/calibration/left.yaml` and `right.yaml`, and restart stereo_vision. Hold the board still at each position, including out in the corners.
- The first build of stereo_vision rebuilds libcamera because of the new patch and EGL/GLES dependencies (about 10 minutes).
- On the final robot with normally mounted cameras: set `OMNIMOW_CAMERA_UPSIDE_DOWN=false` and recalibrate.

---

Test board: rafaelwms/ubuntu-26.04.1-dragon-q6a 1.3.0 (Ubuntu 26.04, mainline kernel 7.2.9, GNOME). The stack runs in ROS 2 Jazzy containers. Merged to main (pull requests #2 and #3, branch `test-setup`).

- Removed what isn't installed on the robot: the model test script (`depth_fusion/test_model.py`) and the training/export scripts (`mlops.py`, `export.py`). They live in the training repo.

- **One-click installer:** A single run prepares the board and builds and starts the whole stack. It can also be piped from curl on a fresh board, in which case it clones the repo itself. It is safe to run again.
- **The desktop stays:** No removal of the GUI or snap, no headless boot. Wi-Fi and Bluetooth stay on. Only ModemManager is disabled, because it interferes with the ESP32s' serial ports.
- Detects the user account created on the board (`--user`, the sudo/pkexec user, the desktop session, or the only regular account) instead of assuming `radxa`.
- **Image-independent:** Installs the FastRPC packages the image has, and never replaces an installed NPU runtime with the conflicting package family. Uses the distribution's Docker if get.docker.com doesn't support the release yet.
- NPU access for the user (the groups `fastrpc`, `dmaheap`, `video` and `render`, plus udev rules) and the `cdsprpcd` daemon.
- Performance mode on every boot via a systemd service.
- Builds one image at a time and creates 8 GB of swap on boards with less than 12 GB of RAM. The parallel builds ran out of memory on the 5 GB board. One failing image doesn't stop the others.
- **Runs without the ESP32s:** The micro-ROS agents are in the compose profile `esp32` and are only started when both ESP32s are connected. Serial numbers in the ESP32 udev rule are preserved when the installer is re-run.
- Docker logs rotate (10 MB × 3 per container).
- Portainer CE at `https://<robot>:9443` (`OMNIMOW_PORTAINER`), outside the OmniMow stack.
- Warnings are collected and shown at the end. Everything is logged to `/var/log/omnimow-install.log`.

- The model is installed from the latest GitHub release (`OMNIMOW_MODEL_REPO`, `OMNIMOW_MODEL_ASSET`) during installation. After that, it checks 2 minutes after boot and every `OMNIMOW_MODEL_CHECK_MIN` minutes (systemd timer).
- A new model is swapped in atomically, and depth_fusion loads it without a restart. The previous one is kept as `*.previous`.
- Private repos: GitHub token in `/etc/omnimow/github_token`.
- `--model FILE|URL` installs a model manually. It is kept until a newer release appears.

- **Device tree:** The image's device tree has CAMSS/CCI disabled and no `__symbols__`, so overlays can't be used. `system_setup/camera/install_camera_dtb.sh` merges Radxa's two Camera 8M 219 overlays (CAM2 = right, CAM3 = left) into the UEFI firmware's own device tree and boots it from a separate systemd-boot entry. The original entry is kept as a fallback. A kernel hook repeats this for new kernels, and `--remove` undoes it.
- **libcamera 0.7 in the container,** because Ubuntu 24.04's 0.2 can't drive CAMSS on the mainline kernel. It is built from source with patch 0001, which gives each camera its own CSID/VFE path so both IMX219s can stream at the same time. Previously this failed with `msm_csid0 ... Device or resource busy`.
- An empty `OMNIMOW_CAMERA_FORMAT` lets the camera choose the format, since there is no NV12 on the mainline stack.
- Scaling and conversion in one multi-threaded step in GStreamer (`videoconvertscale`): stereo went from 2 to about 13 FPS.

- Calibration board: A4, 10 × 7 inner corners, 25 mm squares (Mark Hedley Jones' collection).
- Left and right frames are paired within half a measured frame interval instead of a fixed 20 ms. Previously this failed with "No synchronized frames".
- Logs the stereo rate, time per frame and both cameras' frame rates every 10 seconds.

- **NPU in the container:** The image's FastRPC only looks for the DSP shell in fixed directories and has no `/usr/share/qcom/conf.d`. The container now gets the host's `/usr/lib/dsp` and `/usr/share/qcom`, and the board's DSP directory and QNN's skel directory are added to `ADSP_LIBRARY_PATH`. Previously this failed with `openSessionForPriority failed ... 0x80000600`. FastRPC's log is sent to the host journal.
- qai-appbuilder 2.51.40, because 2.50.40 is no longer available on PyPI.
- Decodes models whose detection head is split into several outputs (boxes, class scores and mask coefficients). The output shapes are logged once per model.
- Masks are computed only within their own box. Same result, but takes 6–16 ms instead of 44–90 ms.
- QNN only logs errors, so there are no per-frame timelines. The 10-second log shows inference time and total time per frame.
- Two Fast DDS changes (LARGE_DATA transport and a 64 MB SHM segment) did not help with the frame loss and were rolled back.

- **localization:** FusionCore v0.4.0 is built from the project's own Dockerfile. The prebuilt image only exists for amd64 and broke the whole `docker compose up`.
- **docker-compose.yml:** The obsolete `version` attribute has been removed.

File: stereo_vision/urdf/OmniMower.urdf (robot description, URDF)
Before this commit: robot omnimower, 3 links, 2 joints
Links:
- removed link gps_link
- added link camera_optical_frame
- added link imu_link
Joints:
- removed joint gps_joint
- added joint camera_optical_joint: type fixed, parent camera_link, child camera_optical_frame, origin xyz=0.0 0.0 0.0 rpy=-1.5707963 0.0 -1.5707963
- added joint imu_joint: type fixed, parent base_link, child imu_link, origin xyz=0.0 0.0 0.05 rpy=0.0 0.0 0.0
